Commit message: Refine Xacro model

File: lab7/urdf/rtr_manipulator.xacro (robot description, xacro)
@@ -1,8 +1,8 @@
 <?xml version="1.0"?>
 <robot xmlns:xacro="http://www.ros.org/wiki/xacro" name="rtr_manipulator">
-  <!-- RTR: Revolute (base yaw) – Prismatic (vertical) – Revolute (elbow). -->
-  <xacro:property name="l2" value="0.9"/>
-  <xacro:property name="l3" value="1.0"/>
-  <xacro:property name="width" value="0.08"/>
+  <!-- Refined RTR dimensions -->
+  <xacro:property name="l2" value="1.0"/>
+  <xacro:property name="l3" value="1.1"/>
+  <xacro:property name="width" value="0.10"/>
   <material name="blue"><color rgba="0 0 1 1"/></material>
   <material name="red"><color rgba="1 0 0 1"/></material>
@@ -10,33 +10,40 @@
   <material name="grey"><color rgba="0.7 0.7 0.7 1"/></material>
   <link name="world"/>
-  <!-- Origins chosen so joint variables match the paper FK (no extra vertical offset in theta_2). -->
   <link name="base_link">
     <visual>
-      <origin xyz="0 0 0.05" rpy="0 0 0"/>
-      <geometry><cylinder radius="0.12" length="0.1"/></geometry>
+      <origin xyz="0 0 0.06"/>
+      <geometry><cylinder radius="0.15" length="0.12"/></geometry>
       <material name="grey"/>
     </visual>
+    <collision>
+      <origin xyz="0 0 0.06"/>
+      <geometry><cylinder radius="0.15" length="0.12"/></geometry>
+    </collision>
   </link>
   <joint name="world_to_base" type="fixed">
     <parent link="world"/>
     <child link="base_link"/>
-    <origin xyz="0 0 0" rpy="0 0 0"/>
+    <origin xyz="0 0 0"/>
   </joint>
   <link name="link_yaw">
     <inertial>
-      <origin xyz="0 0 0" rpy="0 0 0"/>
+      <origin xyz="0 0 0"/>
       <mass value="1"/>
       <inertia ixx="0.01" ixy="0" ixz="0" iyy="0.01" iyz="0" izz="0.01"/>
     </inertial>
     <visual>
-      <origin xyz="0 0 0.15" rpy="0 0 0"/>
-      <geometry><cylinder radius="0.06" length="0.3"/></geometry>
+      <origin xyz="0 0 0.18"/>
+      <geometry><cylinder radius="0.07" length="0.36"/></geometry>
       <material name="blue"/>
     </visual>
+    <collision>
+      <origin xyz="0 0 0.18"/>
+      <geometry><cylinder radius="0.07" length="0.36"/></geometry>
+    </collision>
   </link>
   <joint name="joint_theta1" type="revolute">
     <parent link="base_link"/>
     <child link="link_yaw"/>
-    <origin xyz="0 0 0" rpy="0 0 0"/>
+    <origin xyz="0 0 0"/>
     <axis xyz="0 0 1"/>
     <limit lower="-3.14159" upper="3.14159" effort="100" velocity="1.0"/>
@@ -44,18 +51,20 @@
   <link name="link_carriage">
     <inertial>
-      <origin xyz="0 0 0" rpy="0 0 0"/>
+      <origin xyz="0 0 0"/>
       <mass value="1"/>
       <inertia ixx="0.01" ixy="0" ixz="0" iyy="0.01" iyz="0" izz="0.01"/>
     </inertial>
     <visual>
-      <origin xyz="0 0 0" rpy="0 0 0"/>
       <geometry><box size="${width} ${width} ${width}"/></geometry>
       <material name="green"/>
     </visual>
+    <collision>
+      <geometry><box size="${width} ${width} ${width}"/></geometry>
+    </collision>
   </link>
   <joint name="joint_theta2" type="prismatic">
     <parent link="link_yaw"/>
     <child link="link_carriage"/>
-    <origin xyz="0 0 0" rpy="0 0 0"/>
+    <origin xyz="0 0 0"/>
     <axis xyz="0 0 1"/>
     <limit lower="0.0" upper="2.0" effort="200" velocity="0.25"/>
@@ -63,45 +72,62 @@
   <link name="link_upper">
     <inertial>
-      <origin xyz="${l2/2} 0 0" rpy="0 0 0"/>
+      <origin xyz="${l2/2} 0 0"/>
       <mass value="20"/>
       <inertia ixx="0.1" ixy="0" ixz="0" iyy="1" iyz="0" izz="1"/>
     </inertial>
     <visual>
-      <origin xyz="${l2/2} 0 0" rpy="0 0 0"/>
+      <origin xyz="${l2/2} 0 0"/>
       <geometry><box size="${l2} ${width} ${width}"/></geometry>
       <material name="red"/>
     </visual>
+    <collision>
+      <origin xyz="${l2/2} 0 0"/>
+      <geometry><box size="${l2} ${width} ${width}"/></geometry>
+    </collision>
   </link>
   <joint name="fixed_carriage_upper" type="fixed">
     <parent link="link_carriage"/>
     <child link="link_upper"/>
-    <origin xyz="0 0 0" rpy="0 0 0"/>
+    <origin xyz="0 0 0"/>
   </joint>
   <link name="link_forearm">
     <inertial>
-      <origin xyz="${l3/2} 0 0" rpy="0 0 0"/>
+      <origin xyz="${l3/2} 0 0"/>
       <mass value="20"/>
       <inertia ixx="0.1" ixy="0" ixz="0" iyy="1" iyz="0" izz="1"/>
     </inertial>
     <visual>
-      <origin xyz="${l3/2} 0 0" rpy="0 0 0"/>
+      <origin xyz="${l3/2} 0 0"/>
       <geometry><box size="${l3} ${width} ${width}"/></geometry>
       <material name="blue"/>
     </visual>
+    <collision>
+      <origin xyz="${l3/2} 0 0"/>
+      <geometry><box size="${l3} ${width} ${width}"/></geometry>
+    </collision>
   </link>
   <joint name="joint_theta3" type="revolute">
     <parent link="link_upper"/>
     <child link="link_forearm"/>
-    <origin xyz="${l2} 0 0" rpy="0 0 0"/>
+    <origin xyz="${l2} 0 0"/>
     <axis xyz="0 1 0"/>
     <limit lower="-3.14159" upper="3.14159" effort="100" velocity="1.0"/>
   </joint>
-  <link name="tool0"/>
+  <link name="tool0">
+    <visual>
+      <origin xyz="0.05 0 0"/>
+      <geometry><sphere radius="0.05"/></geometry>
+      <material name="green"/>
+    </visual>
+    <collision>
+      <origin xyz="0.05 0 0"/>
+      <geometry><sphere radius="0.05"/></geometry>
+    </collision>
+  </link>
   <joint name="wrist_to_tool0" type="fixed">
     <parent link="link_forearm"/>
     <child link="tool0"/>
-    <origin xyz="${l3} 0 0" rpy="0 0 0"/>
+    <origin xyz="${l3} 0 0"/>
   </joint>
-  <!-- Ignored by joint_state_publisher_gui / classic chain; required for ros2_control bringup. -->
   <ros2_control name="RTRMock" type="system">
     <hardware>
